Commit message: xacro updated and tool changere integration

File: fanuc_cr_35ib/urdf/fanuc_cr_35ib.urdf.xacro (robot description, xacro)
@@ -1,4 +1,5 @@
 <?xml version="1.0"?>
 <robot name="cr_35ib" xmlns:xacro="http://www.ros.org/wiki/xacro">
+ <xacro:macro name="fanuc" params="prefix parent xyz rpy">
     <xacro:arg name="inertia_mode_sim" default="True"/>
     <xacro:if value="$(arg inertia_mode_sim)">
@@ -9,18 +10,11 @@
     </xacro:unless>
     <!-- <xacro:inertia_data inertia_mode_sim="$(arg inertia_mode_sim)"/> -->
-    <material name="black">
-        <color rgba="0.05 0.05 0.05 1"/>
-    </material>
-    <material name="green">
-        <color rgba="0 0.7 0 1"/>
-    </material>
-    <link name="world"/>
-<!-- base Joint and Link 0 -->
-    <joint name="base_joint" type="fixed">
-        <origin rpy="0 0 0" xyz="0 0 0"/>
-        <parent link="world"/>
-        <child link="sensor"/>
-    </joint>
-    <link name="sensor">
+    <!-- base Joint and Link 0 -->
+    <joint name="${prefix}base_joint" type="fixed">
+        <origin rpy="${rpy}" xyz="${xyz}"/>
+        <parent link="${parent}"/>
+        <child link="${prefix}sensor"/>
+    </joint>
+    <link name="${prefix}sensor">
         <visual>
             <origin rpy="0 0 0" xyz="0 0 0"/>
@@ -42,10 +36,10 @@
         </inertial>
     </link>
-    <joint name="base_joint2" type="fixed">
+    <joint name="${prefix}base_joint2" type="fixed">
         <origin rpy="0 0 0" xyz="0 0 0"/>
-        <parent link="world"/>
-        <child link="base"/>
-    </joint>
-    <link name="base">
+        <parent link="${prefix}sensor"/>
+        <child link="${prefix}base"/>
+    </joint>
+    <link name="${prefix}base">
         <visual>
             <origin rpy="0 0 0" xyz="0 0 0"/>
@@ -67,13 +61,13 @@
         </inertial>
     </link>
-<!-- Joint 1 and Link 1 -->
-    <joint name="J1" type="revolute">
+    <!-- Joint 1 and Link 1 -->
+    <joint name="${prefix}J1" type="revolute">
         <origin rpy="0 0 0" xyz="0 0 0.668"/>
-        <parent link="base"/>
-        <child link="link1"/>
+        <parent link="${prefix}base"/>
+        <child link="${prefix}link1"/>
         <axis xyz="0 0 1"/>
         <limit lower="-3.23" upper="3.23" effort="1" velocity="1.0"/>
     </joint>
-    <link name="link1">
+    <link name="${prefix}link1">
         <visual>
             <origin rpy="0 0 0" xyz="0 0 0"/>
@@ -95,10 +89,10 @@
         </inertial>
     </link>
-    <joint name="cover_j1" type="fixed">
+    <joint name="${prefix}cover_j1" type="fixed">
         <origin rpy="0 0 0" xyz="0 0 0"/>
-        <parent link="link1"/>
-        <child link="cover_j1"/>
-    </joint>
-    <link name="cover_j1">
+        <parent link="${prefix}link1"/>
+        <child link="${prefix}cover_j1"/>
+    </joint>
+    <link name="${prefix}cover_j1">
         <visual>
             <origin rpy="0 0 0" xyz="0 0 0"/>
@@ -120,10 +114,10 @@
         </inertial>
     </link>
-    <joint name="rear_cover_j1" type="fixed">
+    <joint name="${prefix}rear_cover_j1" type="fixed">
         <origin rpy="0 0 0" xyz="0 0 0"/>
-        <parent link="link1"/>
-        <child link="rear_cover_j1"/>
-    </joint>
-    <link name="rear_cover_j1">
+        <parent link="${prefix}link1"/>
+        <child link="${prefix}rear_cover_j1"/>
+    </joint>
+    <link name="${prefix}rear_cover_j1">
         <visual>
             <origin rpy="0 0 0" xyz="0 0 0"/>
@@ -145,13 +139,13 @@
         </inertial>
     </link>
-<!-- Joint 2 and Link 2 -->
-    <joint name="J2" type="revolute">
+    <!-- Joint 2 and Link 2 -->
+    <joint name="${prefix}J2" type="revolute">
         <origin rpy="-1.570796 0 0" xyz="0.075 0 0"/>
-        <parent link="link1"/>
-        <child link="link2"/>
+        <parent link="${prefix}link1"/>
+        <child link="${prefix}link2"/>
         <axis xyz="0 0 1"/>
         <limit lower="-1.40" upper="2.36" effort="1" velocity="1.0"/>
     </joint>
-    <link name="link2">
+    <link name="${prefix}link2">
         <visual>
             <origin rpy="0 0 0" xyz="0 0 0"/>
@@ -173,13 +167,13 @@
         </inertial>
     </link>
-<!-- Joint 3 and Link 3 -->
-    <joint name="J3" type="revolute">
+    <!-- Joint 3 and Link 3 -->
+    <joint name="${prefix}J3" type="revolute">
         <origin rpy="3.141529 0 -1.570796" xyz="0 -0.840 0"/>
-        <parent link="link2"/>
-        <child link="link3"/>
+        <parent link="${prefix}link2"/>
+        <child link="${prefix}link3"/>
         <axis xyz="0 0 1"/>
         <limit lower="-2.42" upper="3.49" effort="1" velocity="1.0"/>
     </joint>
-    <link name="link3">
+    <link name="${prefix}link3">
         <visual>
             <origin rpy="0 0 0" xyz="0 0 0"/>
@@ -201,10 +195,10 @@
         </inertial>
     </link>
-    <joint name="cover_j3" type="fixed">
+    <joint name="${prefix}cover_j3" type="fixed">
         <origin rpy="0 0 0" xyz="0 0 0"/>
-        <parent link="link3"/>
-        <child link="cover_j3"/>
-    </joint>
-    <link name="cover_j3">
+        <parent link="${prefix}link3"/>
+        <child link="${prefix}cover_j3"/>
+    </joint>
+    <link name="${prefix}cover_j3">
         <visual>
             <origin rpy="0 0 0" xyz="0 0 0"/>
@@ -226,13 +220,13 @@
         </inertial>
     </link>
-<!-- Joint 4 and Link 4 -->
-    <joint name="J4" type="revolute">
+    <!-- Joint 4 and Link 4 -->
+    <joint name="${prefix}J4" type="revolute">
         <origin rpy="-1.570796 0 0" xyz="0.215 0 0"/>
-        <parent link="link3"/>
-        <child link="link4"/>
+        <parent link="${prefix}link3"/>
+        <child link="${prefix}link4"/>
         <axis xyz="0 0 1"/>
         <limit lower="-3.49" upper="3.49" effort="1" velocity="1.0"/>
     </joint>
-    <link name="link4">
+    <link name="${prefix}link4">
         <visual>
             <origin rpy="0 0 0" xyz="0 0 0"/>
@@ -254,13 +248,13 @@
         </inertial>
     </link>
-<!-- Joint 5 and Link 5 -->
-    <joint name="J5" type="revolute">
+    <!-- Joint 5 and Link 5 -->
+    <joint name="${prefix}J5" type="revolute">
         <origin rpy="1.570796 0 0" xyz="0 0 -0.890"/>
-        <parent link="link4"/>
-        <child link="link5"/>
+        <parent link="${prefix}link4"/>
+        <child link="${prefix}link5"/>
         <axis xyz="0 0 1"/>
         <limit lower="-2.44" upper="2.44" effort="1" velocity="1.0"/>
     </joint>
-    <link name="link5">
+    <link name="${prefix}link5">
         <visual>
             <origin rpy="0 0 0" xyz="0 0 0"/>
@@ -282,13 +276,13 @@
         </inertial>
     </link>
-<!-- Joint 6 and Link 6 -->
-    <joint name="J6" type="revolute">
+    <!-- Joint 6 and Link 6 -->
+    <joint name="${prefix}J6" type="revolute">
         <origin rpy="-1.570796 0 0" xyz="0 0 0"/>
-        <parent link="link5"/>
-        <child link="link6"/>
+        <parent link="${prefix}link5"/>
+        <child link="${prefix}link6"/>
         <axis xyz="0 0 1"/>
         <limit lower="-7.85" upper="7.85" effort="1" velocity="1.0"/>
     </joint>
-    <link name="link6">
+    <link name="${prefix}link6">
         <visual>
             <origin rpy="0 0 0" xyz="0 0 0"/>
@@ -310,10 +304,31 @@
         </inertial>
     </link>
-<!-- TCP -->
-    <joint name="tcp" type="fixed">
+    <!-- TCP -->
+    <joint name="${prefix}tcp" type="fixed">
         <origin rpy="3.141593 0 0" xyz="0 0 -0.090"/>
-        <parent link="link6"/>
-        <child link="tcp"/>
-    </joint>
-    <link name="tcp"/>
+        <parent link="${prefix}link6"/>
+        <child link="${prefix}tcp"/>
+    </joint>
+    <link name="${prefix}tcp"/>
+    <link name="${prefix}tool_changer_cobot_side">
+        <visual>
+            <origin rpy="0 0 0" xyz="0 0 0"/>
+            <geometry>
+                <mesh filename="package://fanuc_cr_35ib/meshes/tool_changer_cobot_side.stl" scale="0.001 0.001 0.001"/>
+            </geometry>
+            <material name="avorio"/>
+        </visual>
+        <collision>
+            <origin rpy="0 0 0" xyz="0 0 0"/>
+            <geometry>
+                <mesh filename="package://fanuc_cr_35ib/meshes/tool_changer_cobot_side.stl" scale="0.001 0.001 0.001"/>
+            </geometry>
+        </collision>
+    </link>
+    <joint name="${prefix}tc_to_t" type="fixed">
+        <origin rpy="0 0 0" xyz="0 0 -0.0925"/>
+        <parent link="${prefix}link6"/>
+        <child link="${prefix}tool_changer_cobot_side"/>
+    </joint>
+ </xacro:macro>
 </robot>

Commit message: backup

File: fanuc_cr_35ib/urdf/fanuc_cr_35ib.urdf.xacro (robot description, xacro)
@@ -317,5 +317,5 @@
                 <mesh filename="package://fanuc_cr_35ib/meshes/tool_changer_cobot_side.stl" scale="0.001 0.001 0.001"/>
             </geometry>
-            <material name="avorio"/>
+            <material name="army_green"/>
         </visual>
         <collision>
@@ -327,5 +327,5 @@
     </link>
     <joint name="${prefix}tc_to_t" type="fixed">
-        <origin rpy="0 0 0" xyz="0 0 -0.0925"/>
+        <origin rpy="0 0 0" xyz="0 0 -0.090"/>
         <parent link="${prefix}link6"/>
         <child link="${prefix}tool_changer_cobot_side"/>

File: id4_batterypack_description/urdf/materials.xacro (robot description, xacro)
@@ -13,4 +13,10 @@
     <color rgba="0 0.7 0 1"/>
   </material>
+  <material name="army_green">
+    <color rgba="${75/255} ${83/255} ${32/255} 1"/>
+  </material>
+  <material name="avorio">
+    <color rgba="${255/255} ${255/255} ${240/255} 1"/>
+  </material>
   <material name="cornflower_blue">
     <color rgba="${100/255} ${149/255} ${237/255} 1"/>

File: scene_description/urdf/central_rack_tools.xacro (robot description, xacro)
@@ -50,5 +50,5 @@
          </geometry>
          <origin xyz="0 0 0" rpy="0 0 0"/>
-         <material name="cornflower_blue"/>
+         <material name="army_green"/>
         </visual>
         <collision>
@@ -70,5 +70,5 @@
          </geometry>
          <origin xyz="0 0 0" rpy="0 0 0"/>
-         <material name="cornflower_blue"/>
+         <material name="army_green"/>
          </visual>
         <collision>

File: scene_description/urdf/rack_tools_dx.xacro (robot description, xacro)
@@ -2,4 +2,5 @@
 <robot xmlns:xacro="http://wiki.ros.org/xacro" name="rack_tools_dx">
   <xacro:macro name="rack_tools_dx" params="parent xyz rpy">
+    <xacro:include filename="$(find scene_description)/urdf/tool4_gripper.xacro"/>
     <link name="rack_tools_dx">
         <visual>
@@ -28,5 +29,5 @@
          </geometry>
          <origin xyz="0 0 0" rpy="0 0 0"/>
-         <material name="cornflower_blue"/>
+         <material name="army_green"/>
         </visual>
         <collision>
@@ -48,5 +49,5 @@
          </geometry>
          <origin xyz="0 0 0" rpy="0 0 0"/>
-         <material name="cornflower_blue"/>
+         <material name="army_green"/>
          </visual>
         <collision>
@@ -62,24 +63,9 @@
         <origin xyz="-0.1177 0.7 1.0305" rpy="0 0 ${pi}"/>
     </joint>
-    <link name="tool4_gripper_dx">
-        <visual>
-         <geometry>
-             <mesh filename="package://scene_description/meshes/tools/tool4_gripper.stl" scale="0.001  0.001 0.001"/>
-         </geometry>
-         <origin xyz="0 0 0" rpy="0 0 0"/>
-         <material name="cornflower_blue"/>
-        </visual>
-        <collision>
-         <geometry>
-            <mesh filename="package://scene_description/meshes/tools/tool4_gripper.stl" scale="0.001  0.001 0.001"/>
-         </geometry>
-         <origin xyz="0 0 0" rpy="0 0 0"/>
-        </collision>
-    </link>
-    <joint name="rack_dx_to_tool4" type="fixed">
-        <parent link="rack_tools_dx"/>
-        <child link="tool4_gripper_dx"/>
-        <origin xyz="-0.1177 0.4 1.0305" rpy="0 0 ${pi}"/>
-    </joint>
+    <xacro:tool4_gripper
+      prefix="1"
+      parent="rack_tools_dx"
+      xyz="-0.1177 0.4 1.0305"
+      rpy="0 0 ${pi}"/>
   </xacro:macro>
 </robot>

File: scene_description/urdf/rack_tools_sx.xacro (robot description, xacro)
@@ -2,4 +2,5 @@
 <robot xmlns:xacro="http://wiki.ros.org/xacro" name="rack_tools_sx">
   <xacro:macro name="rack_tools_sx" params="parent xyz rpy">
+    <xacro:include filename="$(find scene_description)/urdf/tool4_gripper.xacro"/>
     <link name="rack_tools_sx">
         <visual>
@@ -28,5 +29,5 @@
          </geometry>
          <origin xyz="0 0 0" rpy="0 0 0"/>
-         <material name="cornflower_blue"/>
+         <material name="army_green"/>
         </visual>
         <collision>
@@ -48,5 +49,5 @@
          </geometry>
          <origin xyz="0 0 0" rpy="0 0 0"/>
-         <material name="cornflower_blue"/>
+         <material name="army_green"/>
          </visual>
         <collision>
@@ -62,24 +63,9 @@
         <origin xyz="0.1177 0.7 1.0305" rpy="0 0 0"/>
     </joint>
-    <link name="tool4_gripper_sx">
-        <visual>
-         <geometry>
-             <mesh filename="package://scene_description/meshes/tools/tool4_gripper.stl" scale="0.001  0.001 0.001"/>
-         </geometry>
-         <origin xyz="0 0 0" rpy="0 0 0"/>
-         <material name="cornflower_blue"/>
-        </visual>
-        <collision>
-         <geometry>
-            <mesh filename="package://scene_description/meshes/tools/tool4_gripper.stl" scale="0.001  0.001 0.001"/>
-         </geometry>
-         <origin xyz="0 0 0" rpy="0 0 0"/>
-        </collision>
-    </link>
-    <joint name="rack_sx_to_tool4" type="fixed">
-        <parent link="rack_tools_sx"/>
-        <child link="tool4_gripper_sx"/>
-        <origin xyz="0.1177 0.4 1.0305" rpy="0 0 0"/>
-    </joint>
+    <xacro:tool4_gripper
+      prefix="2"
+      parent="rack_tools_sx"
+      xyz="0.1177 0.4 1.0305"
+      rpy="0 0 0"/>
   </xacro:macro>
 </robot>
